File: Hardware/Qwiic_Mux_PCA9846.brd (EAGLE design)
At the start: 25.4 x 25.4 mm, 29 parts, among them U1 PCA9846

Commit message: Routed
Parts:
- added C3, C4: 2.2uF, SparkFun-Capacitors:0402-TIGHT
- added D1: RED, SparkFun-LED:LED-0603
- added I2C, JP0, JP1, JP2, JP3: JUMPER-SMT_3_2-NC_TRACE_SILK, SparkFun-Jumpers:SMT-JUMPER_3_2-NC_TRACE_SILK
- added LED: JUMPER-SMT_2_NC_TRACE_SILK, SparkFun-Jumpers:SMT-JUMPER_2_NC_TRACE_SILK
- added LOGO4: OSHW-LOGOS, SparkFun-Aesthetics:OSHW-LOGO-S
- added R10, R11, R2, R3, R4, R5, R6, R7, R8, R9: 2.2k, SparkFun-Resistors:0402-TIGHT
- added R12: 1k, SparkFun-Resistors:0402-TIGHT
- added R13: 100k, SparkFun-Resistors:0402-TIGHT
- added U$1: SPARKX-LOGO5, SparkX:SPARKX-LARGE
- C1: value 4.7uF -> 2.2uF; device SparkFun-Capacitors:0603 -> SparkFun-Capacitors:0402-TIGHT
- C2: device SparkFun-Capacitors:0603 -> SparkFun-Capacitors:0402-TIGHT
- J7: device SparkFun-Connectors:1X01_NO_SILK -> SparkFun-Connectors:1X02_NO_SILK
- R1: value 10k -> 100k; device SparkFun-Resistors:0603 -> SparkFun-Resistors:0402-TIGHT
- moved LOGO2 17.8 mm to (-5.08, 17.8)
- moved LOGO3 17.8 mm to (-5.08, 7.62)
- moved R1 7.62 mm to (17.8, 16.5), turned to 180 degrees
- moved C2 3.68 mm to (14.1, 16.5), turned to 180 degrees
- moved C1 3.68 mm to (11.3, 16.5), turned to 0 degrees
- moved J7 2.54 mm to (7.62, 24.1), turned to 270 degrees
- moved FD1 0.63 mm to (5.71, 24.1)
- moved FD3 0.63 mm to (5.71, 24.1)
- moved FD2 0.63 mm to (19.7, 1.27)
- moved FD4 0.63 mm to (19.7, 1.27)
- turned ADDR0 to 90 degrees
- turned ADDR2 to 90 degrees
Connections:
- new net N$1: JP0.3, R2.2
- new net N$10: I2C.1, R11.2
- new net N$11: LED.1, R12.2
- new net N$12: D1.A, R12.1
- new net N$2: JP0.1, R3.2
- new net N$3: JP1.3, R4.2
- new net N$4: JP1.1, R5.2
- new net N$5: JP2.3, R6.2
- new net N$6: JP2.1, R7.2
- new net N$7: JP3.3, R8.2
- new net N$8: JP3.1, R9.2
- new net N$9: I2C.3, R10.2
- net !RESET!: now also J7.2, R13.1; no longer J7.1
- net 3.3V: now also C3.1, C4.1, I2C.2, JP0.2, JP1.2, JP2.2, JP3.2, LED.2, R13.2
- net GND: now also C3.2, C4.2, D1.C, J7.1
- net SC0: now also R3.1
- net SC1: now also R5.1
- net SC2: now also R7.1
- net SC3: now also R9.1
- net SCL: now also R11.1
- net SD0: now also R2.1
- net SD1: now also R4.1
- net SD2: now also R6.1
- net SD3: now also R8.1
- net SDA: now also R10.1
Routing:
- net 3.3V: track 0.00 -> 133.7 mm, vias 0 -> 11
- net GND: track 0.00 -> 77.1 mm, vias 0 -> 30
- net SCL: track 0.00 -> 35.6 mm, vias 0 -> 4
- net SDA: track 0.00 -> 32.6 mm, vias 0 -> 2
- net A0: track 0.00 -> 18.4 mm, vias 0 -> 1
- net SC3: track 0.00 -> 13.6 mm
- net !RESET!: track 0.00 -> 12.5 mm, vias 0 -> 2
- net SC1: track 0.00 -> 12.4 mm
- net N$9: track 0.00 -> 11.6 mm, vias 0 -> 1
- net SC0: track 0.00 -> 10.7 mm, vias 0 -> 2
- net N$3: track 0.00 -> 10.7 mm, vias 0 -> 1
- net SD3: track 0.00 -> 10.3 mm
- net N$4: track 0.00 -> 10.0 mm, vias 0 -> 1
- net SD1: track 0.00 -> 9.73 mm
- net SD0: track 0.00 -> 8.75 mm
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Other:
- board text added: "v01"

Commit message: Ready for review
Parts:
- removed LOGO2, LOGO3: QWIIC_LOGO_7MM, SparkFun-Aesthetics:QWIIC_7MM
- added U$10: (no value), output:#2#9
- added U$11: (no value), output:#3#9
- added U$12: (no value), output:#3V3#7
- added U$13: (no value), output:#A0#0
- added U$14: (no value), output:#A1#1
- added U$15: (no value), output:#A2#2
- added U$16: (no value), output:#A3#3
- added U$17: (no value), output:#A4#4
- added U$18, U$19: (no value), output:#GND#7
- added U$2: (no value), output:PWR43214
- added U$21: (no value), output:#SCL#5
- added U$22: (no value), output:#SDA#6
- added U$23: (no value), output:#LED#0
- added U$24: (no value), output:QWIIC_MUX_PCA98461
- added U$25: (no value), output:#I�C#0
- added U$3: (no value), output:043215
- added U$4: (no value), output:10
- added U$5: (no value), output:211
- added U$6: (no value), output:3212
- added U$7: (no value), output:##RST##8
- added U$8: (no value), output:#0#9
- added U$9: (no value), output:#1#9
- LOGO4: value OSHW-LOGOS -> OSHW-LOGOMINI; device SparkFun-Aesthetics:OSHW-LOGO-S -> SparkFun-Aesthetics:OSHW-LOGO-MINI
- U$1: value SPARKX-LOGO5 -> SPARKX-LOGO3; device SparkX:SPARKX-LARGE -> SparkX:SPARKX-SMALL
- moved U$1 28.2 mm to (20.4, 5.71), flipped to the bottom
- moved LOGO4 25.0 mm to (17.8, 2.54)
- moved FRAME1 16.5 mm to (59.7, -14.0)
- moved LOGO1 15.5 mm to (36.8, 47.0)
- moved I2C 1.91 mm to (14.6, 2.54)
Routing:
- net GND: track 77.1 -> 104.2 mm, vias 30 -> 35
- net 3.3V: track 133.7 -> 135.6 mm
- net N$10: track 6.15 -> 4.41 mm
- net N$9: track 11.6 -> 12.9 mm
- net N$3: track 10.7 -> 11.2 mm
Other:
- board text added: "Dimensions in Inches"
- board text added: "Paul Clark"
- board text added: "Thickness: 1.6mm 2 Layers Black Resist White Silk Finish: HASL Lead Free"
