File: Hardware/Qwiic_Mux_PCA9846.sch (EAGLE design)
At the start: 29 parts, among them U1 PCA9846

Commit message: Routed
Parts:
- added C3, C4: 2.2uF, SparkFun-Capacitors:2.2UF-0402_TIGHT-10V-10%-X5R
- added D1: RED, SparkFun-LED:LED-RED0603
- added I2C, JP0, JP1, JP2, JP3: JUMPER-SMT_3_2-NC_TRACE_SILK, SparkFun-Jumpers:JUMPER-SMT_3_2-NC_TRACE_SILK
- added LED: JUMPER-SMT_2_NC_TRACE_SILK, SparkFun-Jumpers:JUMPER-SMT_2_NC_TRACE_SILK
- added LOGO4: OSHW-LOGOS, SparkFun-Aesthetics:OSHW-LOGOS
- added R10, R11, R2, R3, R4, R5, R6, R7, R8, R9: 2.2k, SparkFun-Resistors:2.2KOHM-0402T-1/16W-1%
- added R12: 1k, SparkFun-Resistors:1KOHM-0402T-1/16W-1%
- added R13: 100k, SparkFun-Resistors:100KOHM-0402T-1/16W-1%
- added U$1: SPARKX-LOGO5, SparkX:SPARKX-LOGO5
- C1: value 4.7uF -> 2.2uF; device SparkFun-Capacitors:4.7UF-0603-6.3V-(10%) -> SparkFun-Capacitors:2.2UF-0402_TIGHT-10V-10%-X5R
- C2: device SparkFun-Capacitors:0.1UF-0603-25V-(+80/-20%) -> SparkFun-Capacitors:0.1UF-0402T-6.3V-10%-X7R
- J7: device SparkFun-Connectors:CONN_01PTH_NO_SILK_YES_STOP -> SparkFun-Connectors:CONN_021X02_NO_SILK
- R1: value 10k -> 100k; device SparkFun-Resistors:10KOHM-0603-1/10W-1% -> SparkFun-Resistors:100KOHM-0402T-1/16W-1%
Connections:
- new net N$1: JP0.3, R2.2
- new net N$10: I2C.1, R11.2
- new net N$11: LED.1, R12.2
- new net N$12: D1.A, R12.1
- new net N$2: JP0.1, R3.2
- new net N$3: JP1.3, R4.2
- new net N$4: JP1.1, R5.2
- new net N$5: JP2.3, R6.2
- new net N$6: JP2.1, R7.2
- new net N$7: JP3.3, R8.2
- new net N$8: JP3.1, R9.2
- new net N$9: I2C.3, R10.2
- net !RESET!: now also J7.2, R13.1, U1.!RESET; no longer J7.1, U1.!RST
- net 3.3V: now also C3.1, C4.1, I2C.2, JP0.2, JP1.2, JP2.2, JP3.2, LED.2, R13.2
- net GND: now also C3.2, C4.2, D1.C, J7.1
- net SC0: now also R3.1
- net SC1: now also R5.1
- net SC2: now also R7.1
- net SC3: now also R9.1
- net SCL: now also R11.1
- net SD0: now also R2.1
- net SD1: now also R4.1
- net SD2: now also R6.1
- net SD3: now also R8.1
- net SDA: now also R10.1
Other:
- note added: "CLOSED OPEN OPEN OPEN CLOSED OPEN OPEN OPEN"
- note added: "LED"
- note added: "OPEN CLOSED OPEN OPEN OPEN CLOSED OPEN OPEN"
- note added: "OPEN OPEN CLOSED OPEN OPEN OPEN CLOSED OPEN"
- note added: "OPEN OPEN OPEN CLOSED OPEN OPEN OPEN CLOSED"
- note added: "OPEN OPEN OPEN OPEN CLOSED CLOSED CLOSED CLOSED"
- note added: "VDD Max: 3.6V VDD Min: 1.65V"
- note removed: "CLOSE OPEN OPEN OPEN CLOSE OPEN OPEN OPEN"
- note removed: "OPEN CLOSE OPEN OPEN OPEN CLOSE OPEN OPEN"
- note removed: "OPEN OPEN CLOSE OPEN OPEN OPEN CLOSE OPEN"
- note removed: "OPEN OPEN OPEN CLOSE OPEN OPEN OPEN CLOSE"
- note removed: "OPEN OPEN OPEN OPEN CLOSE CLOSE CLOSE CLOSE"
- moved on the sheet: ADDR0, ADDR1, ADDR2, ADDR3, ADDR4, C1, C2, IN, J1, OUT, PORT0, PORT1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

Commit message: Ready for review
Parts:
- removed LOGO2, LOGO3: QWIIC_LOGO_7MM, SparkFun-Aesthetics:QWIIC_LOGO_7MM
- LOGO4: value OSHW-LOGOS -> OSHW-LOGOMINI; device SparkFun-Aesthetics:OSHW-LOGOS -> SparkFun-Aesthetics:OSHW-LOGOMINI
- U$1: value SPARKX-LOGO5 -> SPARKX-LOGO3; device SparkX:SPARKX-LOGO5 -> SparkX:SPARKX-LOGO3
Other:
- moved on the sheet: C3, C4, I2C, R10, R11
